File: osprette.kicad_pcb (KiCad board)
At the start: 2 copper layers, 70 parts, among them SW1 SW_Push, SW10 SW_Push, SW11 SW_Push, SW12 SW_Push, SW13 SW_Push, SW14 SW_Push, SW15 SW_Push, SW16 SW_Push, SW17 SW_Push, SW18 SW_Push, SW19 SW_Push, SW2 SW_Push, SW20 SW_Push, SW21 SW_Push, SW22 SW_Push, SW23 SW_Push, SW24 SW_Push, SW25 SW_Push, SW26 SW_Push, SW27 SW_Push, SW28 SW_Push, SW29 SW_Push, SW3 SW_Push, SW30 SW_Push, SW31 SW_Push, SW32 SW_Push, SW33 SW_Push, SW34 SW_Push, SW35 SW_Push, SW4 SW_Push, SW5 SW_Push, SW6 SW_Push, SW7 SW_Push, SW8 SW_Push, SW9 SW_Push, U1 ProMicro_r

Commit message: finalize design, add silk
Parts:
- removed the D14 at (101.8, 91.3)
- removed the SW13 at (86.5, 72.0)
- removed the SW14 at (99.9, 86.0)
- added +: MountingHole_Pad, kbd:1pin_conn, F.Cu at (141.7, 96.9)
- added -: MountingHole_Pad, kbd:1pin_conn, F.Cu at (155.7, 96.9)
- added D5: 1N4148, Diode_SMD:D_SOD-123, B.Cu at (129.1, 92.5)
- added G***: LOGO, Symbol:osprey, F.Cu at (167.5, 121.0)
- added G***: LOGO, Symbol:osprey_flipped, F.Cu at (130.0, 121.0)
- added Ref**: Val**, kbd:M2_HOLE_v3, F.Cu at (201.4, 123.4)
- added Ref**: Val**, kbd:M2_HOLE_v3, F.Cu at (57.2, 79.0)
- added Ref**: Val**, kbd:M2_HOLE_v3, F.Cu at (240.5, 78.9)
- added Ref**: Val**, kbd:M2_HOLE_v3, F.Cu at (182.1, 91.0)
- added Ref**: Val**, kbd:M2_HOLE_v3, F.Cu at (28.0, 99.4)
- added Ref**: Val**, kbd:M2_HOLE_v3, F.Cu at (115.3, 91.3)
- added Ref**: Val**, kbd:M2_HOLE_v3, F.Cu at (269.6, 99.5)
- added Ref**: Val**, kbd:M2_HOLE_v3, F.Cu at (96.1, 123.4)
- added SW31: SW_Push, keyswitches:Kailh_socket_PG1350_optional, F.Cu at (105.6, 133.5)
- added SW36: SW_SPDT, Button_Switch_SMD:SW_SPDT_PCM12, B.Cu at (148.7, 97.9)
- added SW5: SW_Push, keyswitches:Kailh_socket_PG1350_optional, F.Cu at (127.1, 87.3)
- D1, D15, D28: moved to B.Cu
- D10: renamed from D32; moved to B.Cu
- D11: renamed from D2; moved to B.Cu
- D12: renamed from D5; moved to B.Cu
- D13: renamed from D8; moved to B.Cu
- D14: renamed from D11; moved to B.Cu
- D16: renamed from D19; moved to B.Cu
- D17: renamed from D23; moved to B.Cu
- D18: renamed from D27; moved to B.Cu
- D19: renamed from D30; moved to B.Cu
- D2: renamed from D4; moved to B.Cu
- D20: renamed from D33; moved to B.Cu
- D21: renamed from D3; moved to B.Cu
- D22: renamed from D6; moved to B.Cu
- D23: renamed from D9; moved to B.Cu
- D24: renamed from D12; moved to B.Cu
- D25: renamed from D16; moved to B.Cu
- D26: renamed from D20; moved to B.Cu
- D27: renamed from D24; moved to B.Cu
- D29: renamed from D31; moved to B.Cu
- D3: renamed from D7; moved to B.Cu
- D30: renamed from D34; moved to B.Cu
- D31: renamed from D13; moved to B.Cu
- D32: renamed from D17; moved to B.Cu
- D33: renamed from D21; moved to B.Cu
- D34: renamed from D25; moved to B.Cu
- D4: renamed from D10; moved to B.Cu
- D6: renamed from D18; moved to B.Cu
- D7: renamed from D22; moved to B.Cu
- D8: renamed from D26; moved to B.Cu
- D9: renamed from D29; moved to B.Cu
- moved D10 162.2 mm to (274.6, 88.2), turned to 25 degrees
- moved SW10 157.9 mm to (269.3, 86.3), turned to 25 degrees
- moved D4 157.9 mm to (112.8, 85.0), turned to -25 degrees
- moved SW4 154.4 mm to (110.8, 79.7), turned to -25 degrees
- moved D33 148.9 mm to (180.9, 142.9), turned to 25 degrees
- moved SW33 146.8 mm to (175.6, 140.9), turned to 25 degrees
- moved D23 142.7 mm to (85.0, 101.9), turned to -25 degrees
- moved D29 139.1 mm to (239.0, 97.1), turned to 25 degrees
- moved SW23 138.4 mm to (83.1, 96.5), turned to -25 degrees
- moved SW29 135.1 mm to (233.7, 95.1), turned to 25 degrees
- moved D7 130.4 mm to (192.0, 81.5), turned to 25 degrees
- moved SW7 126.8 mm to (186.7, 79.5), turned to 25 degrees
- moved D17 118.0 mm to (199.2, 96.9), turned to 25 degrees
- moved SW17 114.8 mm to (193.9, 94.9), turned to 25 degrees
- moved D13 112.6 mm to (92.2, 86.4), turned to -25 degrees
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- renumbered SW32 to SW10, SW2 to SW11, SW5 to SW12, SW8 to SW13, SW11 to SW14, SW19 to SW16, SW23 to SW17, SW27 to SW18, SW30 to SW19, SW4 to SW2, SW33 to SW20, SW3 to SW21, SW6 to SW22, SW9 to SW23, SW12 to SW24, SW16 to SW25, SW20 to SW26, SW24 to SW27, SW31 to SW29, SW7 to SW3, SW34 to SW30, SW17 to SW32, SW21 to SW33, SW25 to SW34, SW10 to SW4, SW18 to SW6, SW22 to SW7, SW26 to SW8, SW29 to SW9
Connections:
- U1 pad 24: unconnected-(U1-Pad24) -> raw
Routing:
- net row_0: track 0.00 -> 482.4 mm, vias 0 -> 4
- net row_2: track 0.00 -> 404.9 mm, vias 0 -> 3
- net row_1: track 0.00 -> 387.9 mm, vias 0 -> 5
- net col_9: track 0.00 -> 168.9 mm, vias 0 -> 2
- net col_0: track 0.00 -> 156.2 mm
- net row_3: track 0.00 -> 154.0 mm
- net col_8: track 0.00 -> 145.1 mm, vias 0 -> 2
- net col_1: track 0.00 -> 135.5 mm
- net col_7: track 0.00 -> 124.1 mm
- net col_6: track 0.00 -> 119.2 mm, vias 0 -> 4
- net col_2: track 0.00 -> 118.5 mm
- net col_3: track 0.00 -> 117.3 mm, vias 0 -> 2
- net col_5: track 0.00 -> 116.1 mm, vias 0 -> 4
- net col_4: track 0.00 -> 105.3 mm, vias 0 -> 2
- net gnd: track 0.00 -> 53.7 mm, vias 0 -> 1
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- added copper zone on B.Cu, net gnd
- added copper zone on F.Cu, net gnd
Other:
- board outline added: 266.8 x 103.7 mm
