File: osprette.kicad_sch (KiCad schematic)
At the start: 70 parts, among them SW1 SW_Push, SW10 SW_Push, SW11 SW_Push, SW12 SW_Push, SW13 SW_Push, SW14 SW_Push, SW15 SW_Push, SW16 SW_Push, SW17 SW_Push, SW18 SW_Push, SW19 SW_Push, SW2 SW_Push, SW20 SW_Push, SW21 SW_Push, SW22 SW_Push, SW23 SW_Push, SW24 SW_Push, SW25 SW_Push, SW26 SW_Push, SW27 SW_Push, SW28 SW_Push, SW29 SW_Push, SW3 SW_Push, SW30 SW_Push, SW31 SW_Push, SW32 SW_Push, SW33 SW_Push, SW34 SW_Push, SW35 SW_Push, SW4 SW_Push, SW5 SW_Push, SW6 SW_Push, SW7 SW_Push, SW8 SW_Push, SW9 SW_Push, U1 ProMicro_r

Commit message: finalize design, add silk
Parts:
- added +1, -1: MountingHole_Pad, kbd:1pin_conn, symbol Mechanical:MountingHole_Pad
- added SW36: SW_SPDT, Button_Switch_SMD:SW_SPDT_PCM12, symbol Switch:SW_SPDT
- renumbered D32 to D10, D2 to D11, D5 to D12, D8 to D13, D11 to D14, D19 to D16, D23 to D17, D27 to D18, D30 to D19, D4 to D2, D33 to D20, D3 to D21, D6 to D22, D9 to D23, D12 to D24, D16 to D25, D20 to D26, D24 to D27, D31 to D29, D7 to D3, D34 to D30, D13 to D31, D17 to D32, D21 to D33, D25 to D34, D10 to D4, D14 to D5, D18 to D6, D22 to D7, D26 to D8, D29 to D9, SW32 to SW10, SW2 to SW11, SW5 to SW12, SW8 to SW13, SW11 to SW14, SW19 to SW16, SW23 to SW17, SW27 to SW18, SW30 to SW19, SW4 to SW2, SW33 to SW20, SW3 to SW21, SW6 to SW22, SW9 to SW23, SW12 to SW24, SW16 to SW25, SW20 to SW26, SW24 to SW27, SW31 to SW29, SW7 to SW3, SW34 to SW30, SW13 to SW31, SW17 to SW32, SW21 to SW33, SW25 to SW34, SW10 to SW4, SW14 to SW5, SW18 to SW6, SW22 to SW7, SW26 to SW8, SW29 to SW9
Connections:
- net GND: now also -1.1
- net raw: now reaches U1.24 (RAW)
- net raw: now also SW36.3 (C)
- new net bat+: +1.1, SW36.2 (B)
- no-connect marks 6 -> 5
