File: pcb/osprette.kicad_pcb (KiCad board)
At the start: 2 copper layers, 266.8 x 103.7 mm, 83 parts, among them SW1 SW_Push, SW10 SW_Push, SW11 SW_Push, SW12 SW_Push, SW13 SW_Push, SW14 SW_Push, SW15 SW_Push, SW16 SW_Push, SW17 SW_Push, SW18 SW_Push, SW19 SW_Push, SW2 SW_Push, SW20 SW_Push, SW21 SW_Push, SW22 SW_Push, SW23 SW_Push, SW24 SW_Push, SW25 SW_Push, SW26 SW_Push, SW27 SW_Push, SW28 SW_Push, SW29 SW_Push, SW3 SW_Push, SW30 SW_Push, SW31 SW_Push, SW32 SW_Push, SW33 SW_Push, SW34 SW_Push, SW35 SW_Push, SW36 SW_SPDT, SW4 SW_Push, SW5 SW_Push, SW6 SW_Push, SW7 SW_Push, SW8 SW_Push, SW9 SW_Push, U1 ProMicro_r

Commit message: Add (many!) GND vias, to expand copper pours
Routing:
- net reset: track 31.4 -> 32.5 mm
- net gnd: vias 1 -> 64
Changed lines of the file:
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@@
-(kicad_pcb (version 20210824) (generator pcbnew)
+(kicad_pcb (version 20210925) (generator pcbnew)
   (general
     (thickness 1.6)
@@
       (usegerberattributes true)
       (usegerberadvancedattributes true)
-      (creategerberjobfile true)
+      (creategerberjobfile false)
       (svguseinch false)
       (svgprecision 6)
@@
       (plotinvisibletext false)
       (sketchpadsonfab false)
-      (subtractmaskfromsilk false)
+      (subtractmaskfromsilk true)
       (outputformat 1)
       (mirror false)
@@
   (segment (start 137.611641 127.85586) (end 133.174146 137.372092) (width 0.25) (layer "B.Cu") (net 48))
   (segment (start 164.870161 136.595108) (end 160.855289 127.985184) (width 0.25) (layer "B.Cu") (net 48))
-  (segment (start 145.568823 105.122299) (end 145.206501 104.759976) (width 0.25) (layer "F.Cu") (net 49))
-  (segment (start 145.568821 127.622299) (end 145.568823 105.122299) (width 0.25) (layer "F.Cu") (net 49))
+  (segment (start 146.9136 126.27752) (end 146.9136 106.467076) (width 0.25) (layer "F.Cu") (net 49))
+  (segment (start 145.568821 127.622299) (end 146.9136 126.27752) (width 0.25) (layer "F.Cu") (net 49))
   (segment (start 145.206501 104.759976) (end 141.129915 104.75998) (width 0.25) (layer "F.Cu") (net 49))
+  (segment (start 146.9136 106.467076) (end 145.206501 104.759976) (width 0.25) (layer "F.Cu") (net 49))
   (via (at 145.568821 127.622299) (size 0.8) (drill 0.4) (layers "F.Cu" "B.Cu") (net 49))
   (segment (start 145.488514 131.932977) (end 145.488517 127.702606) (width 0.25) (layer "B.Cu") (net 49))
@@
   (segment (start 156.349917 107.299974) (end 156.349915 104.759976) (width 0.25) (layer "F.Cu") (net 50))
   (segment (start 152.891146 107.299976) (end 152.068819 108.122299) (width 0.25) (layer "F.Cu") (net 50))
+  (via (at 158.0388 124.968) (size 0.8) (drill 0.4) (layers "F.Cu" "B.Cu") (free) (net 50))
+  (via (at 108.331 121.3866) (size 0.8) (drill 0.4) (layers "F.Cu" "B.Cu") (free) (net 50))
+  (via (at 102.6922 135.001) (size 0.8) (drill 0.4) (layers "F.Cu" "B.Cu") (free) (net 50))
+  (via (at 165.1 86.8172) (size 0.8) (drill 0.4) (layers "F.Cu" "B.Cu") (free) (net 50))
+  (via (at 166.9542 90.5764) (size 0.8) (drill 0.4) (layers "F.Cu" "B.Cu") (free) (net 50))
+  (via (at 143.002 124.7648) (size 0.8) (drill 0.4) (layers "F.Cu" "B.Cu") (free) (net 50))
+  (via (at 122.8598 105.0798) (size 0.8) (drill 0.4) (layers "F.Cu" "B.Cu") (free) (net 50))
+  (via (at 182.0418 116.8654) (size 0.8) (drill 0.4) (layers "F.Cu" "B.Cu") (free) (net 50))
+  (via (at 117.0686 103.8098) (size 0.8) (drill 0.4) (layers "F.Cu" "B.Cu") (free) (net 50))
+  (via (at 214.249 101.854) (size 0.8) (drill 0.4) (layers "F.Cu" "B.Cu") (free) (net 50))
+  (via (at 186.4868 84.9884) (size 0.8) (drill 0.4) (layers "F.Cu" "B.Cu") (free) (net 50))
+  (via (at 230.7082 93.726) (size 0.8) (drill 0.4) (layers "F.Cu" "B.Cu") (free) (net 50))
+  (via (at 242.6716 91.0844) (size 0.8) (drill 0.4) (layers "F.Cu" "B.Cu") (free) (net 50))
+  (via (at 143.891 97.5868) (size 0.8) (drill 0.4) (layers "F.Cu" "B.Cu") (free) (net 50))
+  (via (at 66.8528 97.6122) (size 0.8) (drill 0.4) (layers "F.Cu" "B.Cu") (free) (net 50))
+  (via (at 233.426 100.6348) (size 0.8) (drill 0.4) (layers "F.Cu" "B.Cu") (free) (net 50))
+  (via (at 115.8494 119.9134) (size 0.8) (drill 0.4) (layers "F.Cu" "B.Cu") (free) (net 50))
+  (via (at 117.5512 144.4244) (size 0.8) (drill 0.4) (layers "F.Cu" "B.Cu") (free) (net 50))
+  (via (at 148.7932 107.2896) (size 0.8) (drill 0.4) (layers "F.Cu" "B.Cu") (free) (net 50))
+  (via (at 122.3772 113.2078) (size 0.8) (drill 0.4) (layers "F.Cu" "B.Cu") (free) (net 50))
+  (via (at 244.1194 98.1964) (size 0.8) (drill 0.4) (layers "F.Cu" "B.Cu") (free) (net 50))
+  (via (at 145.034 100.0506) (size 0.8) (drill 0.4) (layers "F.Cu" "B.Cu") (free) (net 50))
+  (via (at 102.616 92.1004) (size 0.8) (drill 0.4) (layers "F.Cu" "B.Cu") (free) (net 50))
+  (via (at 126.873 135.9662) (size 0.8) (drill 0.4) (layers "F.Cu" "B.Cu") (free) (net 50))
+  (via (at 204.3938 79.4766) (size 0.8) (drill 0.4) (layers "F.Cu" "B.Cu") (free) (net 50))
+  (via (at 111.76 115.3922) (size 0.8) (drill 0.4) (layers "F.Cu" "B.Cu") (free) (net 50))
+  (via (at 78.7654 99.8982) (size 0.8) (drill 0.4) (layers "F.Cu" "B.Cu") (free) (net 50))
+  (via (at 70.3326 76.9366) (size 0.8) (drill 0.4) (layers "F.Cu" "B.Cu") (free) (net 50))
+  (via (at 122.7836 90.6018) (size 0.8) (drill 0.4) (layers "F.Cu" "B.Cu") (free) (net 50))
+  (via (at 92.1258 113.8174) (size 0.8) (drill 0.4) (layers "F.Cu" "B.Cu") (free) (net 50))
+  (via (at 191.1096 93.6244) (size 0.8) (drill 0.4) (layers "F.Cu" "B.Cu") (free) (net 50))
+  (via (at 62.8396 85.1408) (size 0.8) (drill 0.4) (layers "F.Cu" "B.Cu") (free) (net 50))
   (via (at 152.068823 127.622298) (size 0.8) (drill 0.4) (layers "F.Cu" "B.Cu") (net 50))
+  (via (at 174.2948 106.0958) (size 0.8) (drill 0.4) (layers "F.Cu" "B.Cu") (free) (net 50))
+  (via (at 219.075 69.7992) (size 0.8) (drill 0.4) (layers "F.Cu" "B.Cu") (free) (net 50))
+  (via (at 106.2228 83.0072) (size 0.8) (drill 0.4) (layers "F.Cu" "B.Cu") (free) (net 50))
+  (via (at 236.601 93.1418) (size 0.8) (drill 0.4) (layers "F.Cu" "B.Cu") (free) (net 50))
+  (via (at 122.047 101.1428) (size 0.8) (drill 0.4) (layers "F.Cu" "B.Cu") (free) (net 50))
+  (via (at 211.8614 94.7166) (size 0.8) (drill 0.4) (layers "F.Cu" "B.Cu") (free) (net 50))
+  (via (at 175.0314 101.1174) (size 0.8) (drill 0.4) (layers "F.Cu" "B.Cu") (free) (net 50))
+  (via (at 202.4888 117.348) (size 0.8) (drill 0.4) (layers "F.Cu" "B.Cu") (free) (net 50))
+  (via (at 59.4868 98.6028) (size 0.8) (drill 0.4) (layers "F.Cu" "B.Cu") (free) (net 50))
+  (via (at 139.4206 125.2982) (size 0.8) (drill 0.4) (layers "F.Cu" "B.Cu") (free) (net 50))
+  (via (at 115.6208 106.045) (size 0.8) (drill 0.4) (layers "F.Cu" "B.Cu") (free) (net 50))
+  (via (at 234.0864 85.1154) (size 0.8) (drill 0.4) (layers "F.Cu" "B.Cu") (free) (net 50))
+  (via (at 223.774 78.105) (size 0.8) (drill 0.4) (layers "F.Cu" "B.Cu") (free) (net 50))
+  (via (at 99.0854 98.4758) (size 0.8) (drill 0.4) (layers "F.Cu" "B.Cu") (free) (net 50))
+  (via (at 258.0894 93.1672) (size 0.8) (drill 0.4) (layers "F.Cu" "B.Cu") (free) (net 50))
+  (via (at 51.181 86.4362) (size 0.8) (drill 0.4) (layers "F.Cu" "B.Cu") (free) (net 50))
+  (via (at 172.2628 102.5398) (size 0.8) (drill 0.4) (layers "F.Cu" "B.Cu") (free) (net 50))
+  (via (at 148.8186 109.8042) (size 0.8) (drill 0.4) (layers "F.Cu" "B.Cu") (free) (net 50))
+  (via (at 226.2886 85.1916) (size 0.8) (drill 0.4) (layers "F.Cu" "B.Cu") (free) (net 50))
+  (via (at 188.3918 117.1194) (size 0.8) (drill 0.4) (layers "F.Cu" "B.Cu") (free) (net 50))
+  (via (at 157.9118 121.8438) (size 0.8) (drill 0.4) (layers "F.Cu" "B.Cu") (free) (net 50))
+  (via (at 268.986 92.9132) (size 0.8) (drill 0.4) (layers "F.Cu" "B.Cu") (free) (net 50))
+  (via (at 148.8186 112.1918) (size 0.8) (drill 0.4) (layers "F.Cu" "B.Cu") (free) (net 50))
+  (via (at 95.4024 107.569) (size 0.8) (drill 0.4) (layers "F.Cu" "B.Cu") (free) (net 50))
+  (via (at 191.7192 138.7856) (size 0.8) (drill 0.4) (layers "F.Cu" "B.Cu") (free) (net 50))
+  (via (at 177.165 109.5756) (size 0.8) (drill 0.4) (layers "F.Cu" "B.Cu") (free) (net 50))
+  (via (at 89.535 78.3082) (size 0.8) (drill 0.4) (layers "F.Cu" "B.Cu") (free) (net 50))
+  (via (at 179.1462 117.1448) (size 0.8) (drill 0.4) (layers "F.Cu" "B.Cu") (free) (net 50))
+  (via (at 193.6242 100.4316) (size 0.8) (drill 0.4) (layers "F.Cu" "B.Cu") (free) (net 50))
+  (via (at 148.7424 96.901) (size 0.8) (drill 0.4) (layers "F.Cu" "B.Cu") (free) (net 50))
+  (via (at 170.0784 94.2848) (size 0.8) (drill 0.4) (layers "F.Cu" "B.Cu") (free) (net 50))
   (segment (start 154.568823 102.97888) (end 154.568822 102.622297) (width 0.25) (layer "B.Cu") (net 50))
   (segment (start 151.988517 127.702607) (end 152.068823 127.622298) (width 0.25) (layer "B.Cu") (net 50))
